Commit message: feat: use the odom plugin for odometrie

File: robot_indoor/description/robot.urdf.xacro (robot description, xacro)
@@ -4,4 +4,5 @@
     <xacro:include filename="lidar.xacro" />
     <xacro:include filename="camera.xacro" />
+    <xacro:include filename="odom.xacro" />
     <!-- <xacro:include filename="gps.xacro" /> -->
     <xacro:include filename="gazebo_control_04.xacro" />

File: robot_indoor/description/robot_core_04.xacro (robot description, xacro)
@@ -36,5 +36,5 @@
         <parent link="base_link"/>
         <child link="base_footprint"/>
-        <origin xyz="0 0 0" rpy="0 0 0"/>
+        <origin xyz="0 0 ${wheel_offset_z}" rpy="0 0 0"/>
     </joint>
     <link name="base_footprint">
@@ -80,5 +80,5 @@
             <collision>
                 <geometry>
-                    <sphere radius="${wheel_radius}"/>
+                    <cylinder radius="${wheel_radius}" length="${wheel_thickness}"/>
                 </geometry>
             </collision>
